File: platine/platine.kicad_pcb (KiCad board)
At the start: 2 copper layers, 66 x 43.2 mm, 17 parts, among them J1 Screw_Terminal_01x02, J2 Screw_Terminal_01x02, J3 Screw_Terminal_01x02, Q1 BC547, Q2 BC337, SW1 SW_Push_Dual, U1 ATtiny13A-PU

Commit message: small optimisations on PCB
Parts:
- moved J1 2.54 mm to (88.9, 121.9)
Routing:
- net +5V: track 167.4 -> 163.8 mm
- net GND: track 161.0 -> 158.4 mm
Other:
- board size 66 x 43.2 mm -> 66 x 40.6 mm
Changed lines of the file:
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@@
     (thickness 1.6)
     (drawings 4)
-    (tracks 111)
+    (tracks 109)
     (zones 0)
     (modules 17)
@@
   )
   (module TerminalBlock_Phoenix:TerminalBlock_Phoenix_MKDS-1,5-2-5.08_1x02_P5.08mm_Horizontal (layer F.Cu)
-    (at 88.9 124.46)
+    (at 88.9 121.92)
     (descr "Terminal Block Phoenix MKDS-1,5-2-5.08, 2 pins, pitch 5.08mm, size 10.2x9.8mm^2, drill diamater 1.3mm, pad diameter 2.6mm, see http://www.farnell.com/datasheets/100425.pdf, script-generated using https://github.com/pointhi/kicad-footprint-generator/scripts/TerminalBlock_Phoenix")
     (tags "THT Terminal Block Phoenix MKDS-1,5-2-5.08 pitch 5.08mm size 10.2x9.8mm^2 drill 1.3mm pad 2.6mm")
@@
       (effects (font (size 1 1) (thickness 0.15)))
     )
-    (fp_text value 10K (at 3.81 2.37 90) (layer F.Fab)
+    (fp_text value 10K (at 3.81 -0.508 90) (layer F.Fab)
       (effects (font (size 1 1) (thickness 0.15)))
     )
@@
       (effects (font (size 1 1) (thickness 0.15)))
     )
-    (fp_text value 1K (at 3.81 2.37 90) (layer F.Fab)
+    (fp_text value 1K (at 3.81 -0.508 90) (layer F.Fab)
       (effects (font (size 1 1) (thickness 0.15)))
     )
@@
       (effects (font (size 1 1) (thickness 0.15)))
     )
-    (fp_text value 1K (at 3.81 2.37 90) (layer F.Fab)
+    (fp_text value 1K (at 3.81 0 90) (layer F.Fab)
       (effects (font (size 1 1) (thickness 0.15)))
     )
@@
       (effects (font (size 1 1) (thickness 0.15)))
     )
-    (fp_text value 220 (at 3.81 2.37) (layer F.Fab)
+    (fp_text value 220 (at 3.81 0) (layer F.Fab)
       (effects (font (size 1 1) (thickness 0.15)))
     )
@@
       (effects (font (size 1 1) (thickness 0.15)))
     )
-    (fp_text value 220 (at 3.81 2.37) (layer F.Fab)
+    (fp_text value 220 (at 3.81 0) (layer F.Fab)
       (effects (font (size 1 1) (thickness 0.15)))
     )
@@
       (effects (font (size 1 1) (thickness 0.15)))
     )
-    (fp_text value 220 (at 3.81 2.37) (layer F.Fab)
+    (fp_text value 220 (at 3.81 0) (layer F.Fab)
       (effects (font (size 1 1) (thickness 0.15)))
     )
@@
   )
   (gr_line (start 129.54 88.9) (end 63.5 88.9) (layer Edge.Cuts) (width 0.15))
-  (gr_line (start 129.54 132.08) (end 129.54 88.9) (layer Edge.Cuts) (width 0.15))
-  (gr_line (start 63.5 132.08) (end 129.54 132.08) (layer Edge.Cuts) (width 0.15))
-  (gr_line (start 63.5 88.9) (end 63.5 132.08) (layer Edge.Cuts) (width 0.15))
+  (gr_line (start 129.54 129.54) (end 129.54 88.9) (layer Edge.Cuts) (width 0.15))
+  (gr_line (start 63.5 129.54) (end 129.54 129.54) (layer Edge.Cuts) (width 0.15))
+  (gr_line (start 63.5 88.9) (end 63.5 129.54) (layer Edge.Cuts) (width 0.15))
   (segment (start 85.01 100.25) (end 86.36 101.6) (width 0.4) (layer B.Cu) (net 1))
   (segment (start 81.28 100.25) (end 85.01 100.25) (width 0.4) (layer B.Cu) (net 1))
@@
   (segment (start 71.04 124.38) (end 81.28 124.38) (width 0.4) (layer B.Cu) (net 3))
   (segment (start 66.04 119.38) (end 71.04 124.38) (width 0.4) (layer B.Cu) (net 3))
-  (segment (start 101.6 127) (end 101.6 124.46) (width 0.4) (layer B.Cu) (net 3))
-  (segment (start 91.44 127) (end 101.6 127) (width 0.4) (layer B.Cu) (net 3))
-  (segment (start 88.9 124.46) (end 91.44 127) (width 0.4) (layer B.Cu) (net 3))
+  (segment (start 88.9 124.46) (end 101.6 124.46) (width 0.4) (layer B.Cu) (net 3))
   (segment (start 71.12 119.3) (end 68.66 116.84) (width 0.4) (layer B.Cu) (net 4))
   (segment (start 68.66 116.84) (end 68.66 114.38) (width 0.4) (layer B.Cu) (net 4))
@@
   (segment (start 81.28 119.38) (end 93.98 119.38) (width 0.4) (layer B.Cu) (net 4))
   (segment (start 93.98 119.38) (end 93.98 114.808) (width 0.4) (layer B.Cu) (net 4))
-  (segment (start 93.98 124.46) (end 93.98 119.38) (width 0.4) (layer B.Cu) (net 4))
+  (segment (start 93.98 119.38) (end 93.98 121.92) (width 0.4) (layer B.Cu) (net 4))
   (segment (start 123.19 96.52) (end 123.19 105.41) (width 0.4) (layer B.Cu) (net 5))
   (segment (start 119.38 119.38) (end 121.92 116.84) (width 0.4) (layer B.Cu) (net 6))
